Commit message: Update UR20 camera calibration assets

File: ur20_description/ur20_with_camera.urdf (robot description, URDF)
Before this commit: robot ur, 18 links, 17 joints
Joints:
- joint camera_joint: origin xyz=0 -0.03 0.100 rpy=0 1.57 0 -> xyz=0 -0.03 0.100 rpy=0 1.5707963267948966 0
- joint camera_optical_joint: origin xyz=-0.1 0.03 0 rpy=0 -1.57 0 -> xyz=-0.212 0.03 0 rpy=0 -1.5707963267948966 0
