Commit message: fix(camera): camera_optical_frame 을 body_face(0.141)로 이전
CAD(camera_asm_wo_light.stp) 실측 결과 구값 0.346 은 어셈블리에서 제거된
조명박스 LIGHT_1 의 앞면이었다. 프레임을 카메라 몸체 앞면(flange+141.0mm)으로
옮기고 WD 를 250mm 로 맞춰, CAMERA_WORKING_DISTANCE_MM 이 벤더 공칭 WD 와
같은 기준점을 쓰도록 정렬했다.

- 141.0 + 250.0 = 391.0 = CAD VIEW_1(50x50 검사면 판) 근접면
- 물체면은 392 -> 391 로 1mm 만 이동 -> 도달성 회귀 없음
  (sample/74 73/74=98.6%, curved_structure/100 97/100=97.0%)
- 렌더 프러스텀이 focalLength=250, aperture=50 이 되어 CAD 의도와 일치
  (기존 46mm 기준은 꼭짓점이 허공이라 화각 콘이 실제보다 넓었다)

동기화 대상: URDF camera_optical_joint / USD 2개의 camera_optical_frame /
build_camera_mesh.OPTICAL_FRAME_X / config 2개 상수. viewpoint h5 는 재생성했다.
h5 의 working_distance_mm 가 config 를 이기므로, 불일치 시 storage.py 가 경고한다.

파킹 해소: 벤더 WD 250mm 의 기준점은 body_face 였다(78mm 차는 배럴 길이 자체).
검증: 계산된 렌즈 배럴 끝 218.770mm = build_camera_mesh.EXPECT_HI[0] 0.21877m.

docs: robot-camera-assets.md 신규(에셋 소유권 지도 + 동기화 체크리스트),
camera-geometry.md 전면 개정, inspect_camera_step.py 신규(CAD 실측 재현 툴).

Co-Authored-By: Claude Opus 5 (1M context) <noreply@anthropic.com>

File: workcell/robot/ur20_with_camera_curobo.urdf (robot description, URDF)
Before this commit: robot ur, 14 links, 13 joints
Joints:
- joint camera_optical_joint: origin xyz=0.346 0 0 rpy=1.5707963268 -0.0000000000 1.5707963268 -> xyz=0.141 0 0 rpy=1.5707963268 -0.0000000000 1.5707963268

Commit message: fix(camera): 카메라 clocking 을 실기에 맞춰 roll -90deg 로 (URDF+USD)
실로봇과 대조해보니 카메라가 플랜지에 물린 각도가 시뮬과 달랐다. 회전축은 툴
축(flange +X = 광축)이라 광축 방향도 camera_optical_frame 원점(0.141,0,0)도
움직이지 않는다 — 몸체가 어느 쪽으로 뻗는지와 이미지 회전만 바뀐다. FK 로 확인:
flange 좌표 몸체 bbox 가 y[-94.9,+50] z[-56,+56] -> y[-56,+56] z[-50,+94.9] mm.

USD 의 camera_mount 프림은 원래 이 용도로 rotateXYZ 를 들고 있었고(그동안 0),
URDF 의 camera_mount_joint 가 그 짝이다. ghost 는 로봇 USD 에서 재생성했다.
camera_link 충돌 스피어 34개는 그 프레임째 같이 돌아 재피팅이 필요 없다.

verify_composed 의 'mesh->flange identity' assert 는 mount 프레임 기준으로 바꾸고,
URDF rpy <-> USD rotateXYZ <-> CAMERA_MOUNT_RPY_DEG 3자 교차검증을 추가했다 —
한쪽만 고치면 계획(cuRobo)과 화면(USD)이 다른 로봇이 되는데 그동안 아무도 에러를
내지 않았다. 메시가 사는 프레임이 flange 가 아니게 되어 R_NEW_TO_FLANGE ->
R_NEW_TO_MOUNT, assert_flange_bbox -> assert_mount_bbox 로 이름도 정정.

h5 재생성은 불필요하다(viewpoint 위치도 WD 기하도 그대로). 충돌 형상은 실제로
바뀌지만 sample/74 전후 실측은 동일했다: 도달 73/74, 충돌제거 0, 후보 279->275.

문서: 프레임 체인 갱신 + clocking 변경 절차 신설. 겸사겸사 §2 표의 오류도 정정 —
workcell/robot/ur20_with_camera.xrdf 가 "MoveIt/cuMotion launch 가 읽는다"고 돼
있었으나 실제로는 아무도 안 읽는다. MoveIt 은 ur_gated.urdf.xacro(순정 UR20) +
scripts/moveit/ur20.xrdf 를 쓰고 둘 다 카메라가 없다. 별도 과제로 남긴다.

Co-Authored-By: Claude Opus 5 (1M context) <noreply@anthropic.com>

File: workcell/robot/ur20_with_camera_curobo.urdf (robot description, URDF)
Before this commit: robot ur, 14 links, 13 joints
Joints:
- joint camera_mount_joint: origin xyz=0 0 0 rpy=0 0 0 -> xyz=0 0 0 rpy=-1.5707963268 0 0

Commit message: fix(camera): WD 기준점을 카메라 끝(렌즈 배럴 앞면)으로 이전
WD 를 body_face(커버 앞면, flange+141.0mm)에서 쟀는데, 그 점은 CAD 를 파싱해야만
찾을 수 있어 현장에서 자로 확인할 방법이 없었다. camera_optical_frame 을 카메라의
물리적 최전단인 렌즈 배럴 앞면(flange+218.770mm)으로 옮겨, "카메라 끝 → 물체" 가
그대로 코드의 WD 가 되게 했다.

camera_optical_frame 이 곧 WD 기준점이라(tool_frames[0] · poses.build_camera_poses ·
Isaac 프러스텀 꼭짓점) 기준점 변경과 프레임 이동은 같은 작업이다. 프레임을 옮기면
하류 코드는 한 줄도 바뀌지 않는다.

- 검사면은 flange+391.0mm(CAD VIEW_1) 그대로 → WD 250 -> 172.23 으로 상보 조정
  (218.770 + 172.230 = 391.000). 구 기준 값 환산: 새 WD = 구 WD - 77.770
- 로봇 기하 불변 확인: cylinder_sample/132 (WD 273 -> 195.23) 도달성
  118/132 로 변경 전과 **reachable 목록까지 동일**. 후보 수만 362 -> 364
  (multi-seed IK 표본 흔들림)
- CAMERA_MIN_WORKING_DISTANCE_MM 은 77.8 -> 0.0 (수식 lens_front - optical_frame 유지)
- CAMERA_NEAR_CLIP_M 은 기하 파생을 끊고 10mm 고정 — 카메라 원점 앞을 가리는
  자기 부품이 사라져 "배럴 너머로 민다"는 근거 자체가 없어졌다

동기화: URDF camera_optical_joint / USD 2개의 camera_optical_frame 트랜스폼 /
build_camera_mesh.OPTICAL_FRAME_X / config 상수. ghost 는 build_ghost_usd.py 로
재생성했고(구조 diff 결과 의미 차이는 이 트랜스폼 하나뿐), --verify-only --ghost 통과.

⚠️ 기존 h5 는 이번에 손대지 않았다. 250·273 같은 구 기준 값은 새 기준에서도 유효한
숫자라 working_distance_error() 를 그냥 통과하고 검사면만 77.770mm 멀어진다.
후속 작업으로 남긴다(camera-geometry.md §미해결).

Co-Authored-By: Claude Opus 5 (1M context) <noreply@anthropic.com>

File: workcell/robot/ur20_with_camera_curobo.urdf (robot description, URDF)
Before this commit: robot ur, 14 links, 13 joints
Joints:
- joint camera_optical_joint: origin xyz=0.141 0 0 rpy=1.5707963268 -0.0000000000 1.5707963268 -> xyz=0.21877 0 0 rpy=1.5707963268 -0.0000000000 1.5707963268
